File: kicad_docs/oscillator_carrier_board.kicad_pcb (KiCad board)
At the start: 2 copper layers, 68.6 x 99.1 mm, 22 parts, among them J1 1v_per_oct_in, J10 Conn_01x05, J11 Conn_01x04, J12 Conn_01x02, J13 Conn_01x02, J14 Conn_01x05, J15 Conn_01x05, J2 expo_fm_in, J3 lin_fm_in, J4 sync_in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

Commit message: update silkscreen with git info
Other:
- board text added: "https://github.com/JordanAceto/Oscillator_Carrier_Board rev 1 2020-02-02"
Changed lines of the file:
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@@
   (general
     (thickness 1.6)
-    (drawings 19)
+    (drawings 20)
     (tracks 107)
     (zones 0)
@@
     )
   )
+  (gr_text "https://github.com/JordanAceto/Oscillator_Carrier_Board\nrev 1\n2020-02-02" (at 168.91 55.245) (layer B.SilkS)
+    (effects (font (size 1 1) (thickness 0.15)) (justify left mirror))
+  )
   (gr_text "pulse out" (at 161.29 132.715) (layer F.SilkS)
